File: power-management-board/power-management-board.kicad_pcb (KiCad board)
At the start: 2 copper layers, 90 x 70 mm, 118 parts, among them IC1 LM74502QDDFRQ1, IC2 TLP7820_TP4,E, IC3 MCP2562, J1 Conn_01x02, J2 Conn_01x02, J3 Conn_01x04, J4 Conn_01x04, J5 Conn_01x04_Pin, J6 Conn_01x02_Pin, J7 Conn_01x02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

Commit message: 完成(ビア以外)
Parts:
- removed JP2: Jumper_2_Open, Connector_PinHeader_2.54mm:PinHeader_1x02_P2.54mm_Vertical
- added D19: LED, LED_SMD:LED_0603_1608Metric_Pad1.05x0.95mm_HandSolder, F.Cu at (26.9, 18.3)
- added D20: LED, LED_SMD:LED_0603_1608Metric_Pad1.05x0.95mm_HandSolder, F.Cu at (28.6, 18.3)
- added D21: LED, LED_SMD:LED_0603_1608Metric_Pad1.05x0.95mm_HandSolder, F.Cu at (101.8, 46.4)
- added D22: LED, LED_SMD:LED_0603_1608Metric_Pad1.05x0.95mm_HandSolder, F.Cu at (76.0, 52.0)
- added R42: 1k, Resistor_SMD:R_0603_1608Metric_Pad0.98x0.95mm_HandSolder, F.Cu at (26.9, 21.7)
- added R43: 1k, Resistor_SMD:R_0603_1608Metric_Pad0.98x0.95mm_HandSolder, F.Cu at (28.6, 21.7)
- added R44: 1k, Resistor_SMD:R_0603_1608Metric_Pad0.98x0.95mm_HandSolder, F.Cu at (98.4, 46.4)
- added R45: 1k, Resistor_SMD:R_0603_1608Metric_Pad0.98x0.95mm_HandSolder, F.Cu at (74.4, 52.0)
- added SW3: SW_SPDT_312, 0Ikedalibrary:CJS1200A1, F.Cu at (33.8, 20.9)
- J3, J4: footprint Connector_JST:JST_XH_B4B-XH-A_1x04_P2.50mm_Vertical -> Connector_JST:JST_XH_S4B-XH-A_1x04_P2.50mm_Horizontal; moved to B.Cu
- moved R14 26.0 mm to (89.2, 57.8), turned to 90 degrees
- moved R12 22.3 mm to (101.2, 53.6)
- moved R11 22.3 mm to (95.1, 53.6)
- moved R13 22.2 mm to (83.2, 57.8), turned to 90 degrees
- moved F2 21.3 mm to (64.6, 47.6)
- moved C9 20.4 mm to (67.2, 48.5), turned to -90 degrees
- moved C10 20.0 mm to (74.4, 48.6), turned to 90 degrees
- moved U7 19.1 mm to (70.8, 48.5), turned to 0 degrees
- moved R16 17.9 mm to (78.4, 52.0)
- moved C6 17.9 mm to (76.0, 48.6), turned to 90 degrees
- moved C7 17.0 mm to (79.6, 36.0)
- moved R15 16.9 mm to (79.2, 54.8), turned to -90 degrees
- moved IC2 14.3 mm to (80.2, 44.8)
- moved C8 13.3 mm to (79.6, 37.6)
- moved C21 11.7 mm to (38.0, 29.2)
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Connections:
- U2 pad 4: discharge -> GND
- U2 pad 6: GND -> discharge
Routing:
- net discharge: track 0.00 -> 21.4 mm
- net VIN: track 11.6 -> 32.2 mm, vias 0 -> 1
- net +5VA: track 30.5 -> 48.1 mm, vias 0 -> 2
- net Voltage_sensor_VOUT: track 43.4 -> 27.8 mm
- net CANL: track 15.1 -> 26.4 mm
- net VOUT: track 8.88 -> 19.4 mm, vias 0 -> 1
- net CANH: track 15.1 -> 24.2 mm, vias 0 -> 1
- net +3.3V: track 147.4 -> 155.7 mm, vias 9 -> 7
- net IP: track 1.30 -> 6.72 mm, vias 0 -> 2
- net CAN_RX: track 9.48 -> 14.7 mm
- net +5V: track 5.80 -> 10.9 mm
- net stm_discharge: track 46.7 -> 50.2 mm, vias 2 -> 0
- net IN2: track 29.6 -> 26.5 mm
- net Net-(IC2-VIN+): track 7.00 -> 4.05 mm
- net Net-(SW3-A): track 0.00 -> 1.94 mm
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- added copper zone on B.Cu, net GND
- added copper zone on F.Cu, net GND
- added copper zone on B.Cu, net GND1
- added copper zone on F.Cu, net GND1
- added copper zone on B.Cu, net GNDD
- added copper zone on F.Cu, net GNDD
- added copper zone on B.Cu, net IP
- added copper zone on F.Cu, net IP
- added copper zone on F.Cu, net Net-(IC1-SRC)
- added copper zone on B.Cu, net VIN
- added copper zone on F.Cu, net VIN
- added copper zone on B.Cu, net VOUT
- added copper zone on F.Cu, net VOUT
Other:
- board text added: "."
- board text added: "1"
- board text added: "2"
- board text added: "2 1 G"
- board text added: "3"
- board text added: "4"
- board text added: "5V (VSn)"
- board text added: "5V 3.3V"
- board text added: "C"
- board text added: "D"
- board text added: "EN"
- board text added: "EN IN"
- board text added: "EN OUT"
- board text added: "G"
- board text added: "G L 5V H"
- board text added: "I"
- board text added: "IN1"
- board text added: "IN2"
- board text added: "K"
- board text added: "L"
- board text added: "O"
- board text added: "R"
- board text added: "T"
- board text added: "U"
- board text added: "V"
- board text added: "VIN"
- board text added: "c"
- board text added: "h"
- board text added: "駆動系"
- board text removed: "IN2 IN1"
- board text removed: "VCC"
- board text removed: "駆動系 EN"

Commit message: 完成
Parts:
- added G***: LOGO, LOGO, F.Cu at (60.9, 81.6)
- moved C3 19.4 mm to (53.4, 68.5)
- moved C4 19.4 mm to (72.8, 68.5)
- moved J2 0.30 mm to (99.7, 72.0)
- moved R29 0.14 mm to (33.9, 17.1)
Routing:
- net VIN: track 32.2 -> 30.5 mm, vias 1 -> 70
- net CAN_RX: track 14.7 -> 14.0 mm
- net CANH: track 24.2 -> 24.8 mm
- net GND: track 0.04 -> 0.00 mm, vias 32 -> 159
- net VOUT: vias 1 -> 87
- net IP: vias 2 -> 45
- net GNDD: vias 11 -> 113
- net GNDA: vias 4 -> 19
- net GND1: vias 5 -> 39
Other:
- board text added: "power-management-board version 1.0 create by ikeda"
