File: power-management-board/power-management-board.kicad_pcb (KiCad board)
At the start: 2 copper layers, 90 x 70 mm, 127 parts, among them IC1 LM74502QDDFRQ1, IC2 TLP7820_TP4,E, IC3 MCP2562, J1 Conn_01x02, J2 Conn_01x02, J3 Conn_01x04, J4 Conn_01x04, J5 Conn_01x04_Pin, J6 Conn_01x02_Pin, J7 Conn_01x02, J8 Conn_01x02, J9 Conn_01x03, Q1 XPQR8308QB,LXHQ, Q2 XPQR8308QB,LXHQ, SW2 SW_SPDT_312, SW3 SW_SPDT_312, U1 TLP293, U2 TLP3546A, U3 STM32G431K8Tx, U4 NJM12888F33, U5 TLP293, U6 CZ3A07, U7 AP7375, U8 TLP293, U9 TLP293

Commit message: LM74502QDDFRQ1からLTC4368IMS2PBFに変更
Parts:
- removed C1: 0.1uf, Capacitor_SMD:C_0603_1608Metric_Pad1.08x0.95mm_HandSolder
- removed C2: 0.47uf, Capacitor_SMD:C_0603_1608Metric_Pad1.08x0.95mm_HandSolder
- removed D1: MS18F, Diode_SMD:D_2010_5025Metric_Pad1.52x2.65mm_HandSolder
- removed IC1: LM74502QDDFRQ1, Package_TO_SOT_SMD:SOT-23-8_Handsoldering
- removed JP1: Jumper_2_Open, Connector_PinHeader_2.54mm:PinHeader_1x02_P2.54mm_Vertical
- removed R2: 10, Resistor_SMD:R_0603_1608Metric_Pad0.98x0.95mm_HandSolder
- removed R3: 100k 1%, Resistor_SMD:R_0603_1608Metric_Pad0.98x0.95mm_HandSolder
- removed R4: 5.1k 1%, Resistor_SMD:R_0603_1608Metric_Pad0.98x0.95mm_HandSolder
- removed SW2: SW_SPDT_312, 0Ikedalibrary:CJS1200A1
- added C24: 0.22uf, Capacitor_SMD:C_0603_1608Metric_Pad1.08x0.95mm_HandSolder, F.Cu at (27.9, 46.0)
- added C25: 0.1uf, Capacitor_SMD:C_0603_1608Metric_Pad1.08x0.95mm_HandSolder, F.Cu at (27.7, 40.5)
- added C26: 3.3nf, Capacitor_SMD:C_0603_1608Metric_Pad1.08x0.95mm_HandSolder, F.Cu at (31.3, 46.0)
- added D23: CUHS20S60, 0Ikedalibrary:Diode_US2H, F.Cu at (35.0, 42.5)
- added D24: LED, LED_SMD:LED_0603_1608Metric_Pad1.05x0.95mm_HandSolder, F.Cu at (22.1, 40.9)
- added D25: CUHS20S60, 0Ikedalibrary:Diode_US2H, F.Cu at (23.8, 44.9)
- added D26: CUHS20S60, 0Ikedalibrary:Diode_US2H, F.Cu at (22.2, 42.8)
- added D27: CUHS20S60, 0Ikedalibrary:Diode_US2H, F.Cu at (42.3, 42.4)
- added D28: CUHS20S60, 0Ikedalibrary:Diode_US2H, F.Cu at (42.5, 38.6)
- added IC4: LTC4368IMS-2#PBF, 0Ikedalibrary:SOP50P490X110-10N, F.Cu at (29.9, 43.2)
- added R46: 10k, Resistor_SMD:R_0603_1608Metric_Pad0.98x0.95mm_HandSolder, F.Cu at (31.2, 40.5)
- added R47: 10k, Resistor_SMD:R_0603_1608Metric_Pad0.98x0.95mm_HandSolder, F.Cu at (38.6, 42.1)
- added R48: 10k, Resistor_SMD:R_0603_1608Metric_Pad0.98x0.95mm_HandSolder, F.Cu at (34.6, 40.5)
- added R49: 10k, Resistor_SMD:R_0603_1608Metric_Pad0.98x0.95mm_HandSolder, F.Cu at (38.0, 40.5)
- added R51: 10k, Resistor_SMD:R_0603_1608Metric_Pad0.98x0.95mm_HandSolder, F.Cu at (21.1, 45.5)
- added R52: 10k, Resistor_SMD:R_0603_1608Metric_Pad0.98x0.95mm_HandSolder, F.Cu at (39.7, 38.8)
- added R53: 22k, Resistor_SMD:R_0603_1608Metric_Pad0.98x0.95mm_HandSolder, F.Cu at (34.7, 46.0)
- R1: value 10k -> 1k
- moved U1 4.00 mm to (36.5, 36.4), turned to 0 degrees
- moved R1 2.59 mm to (25.1, 42.0), turned to 90 degrees
- renumbered RST to SW1
Connections:
- R1 pad 1: EN -> Net-(D25-Pad1)
- R1 pad 2: GND -> Net-(D24-A)
- U1 pad 4: VIN -> Net-(D27-Pad1)
Routing:
- net Net-(IC1-OV): track 17.0 -> 0.00 mm, vias 2 -> 0
- net Net-(IC4-OV): track 0.00 -> 13.8 mm, vias 0 -> 2
- net Net-(D24-K): track 0.00 -> 11.5 mm, vias 0 -> 2
- net Net-(IC4-UV): track 0.00 -> 11.1 mm, vias 0 -> 2
- net VIN: track 30.5 -> 40.3 mm
- net Net-(D27-Pad1): track 0.00 -> 9.53 mm
- net Net-(D24-A): track 0.00 -> 6.62 mm
- net Net-(D25-Pad1): track 0.00 -> 5.02 mm
- net Net-(Q1-S): track 4.20 -> 0.00 mm
- net EN: track 19.5 -> 15.8 mm
- net Net-(D23-Pad1): track 0.00 -> 3.75 mm
- net Net-(IC4-RETRY): track 0.00 -> 3.65 mm
- net Net-(IC1-VCAP): track 1.86 -> 0.00 mm
- net Net-(C26-Pad2): track 0.00 -> 1.66 mm
- net Net-(C2-Pad2): track 1.60 -> 0.00 mm
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Other:
- board text added: "FAULT"
- board text removed: "常時ON"
- board text removed: "過電圧保護"

Commit message: 抵抗の計算完了、常時ONのジャンパーPINの追加
Parts:
- added JP1: jp, Connector_PinHeader_2.54mm:PinHeader_1x02_P2.54mm_Vertical, F.Cu at (41.4, 44.8)
- C26: value 3.3nf -> 0.1uf
- R46, R49: value 10k -> 2k
- R47: value 10k -> 3k
- R48: value 10k -> 143k
- moved D27 3.00 mm to (42.3, 39.4)
- moved D28 2.90 mm to (42.5, 35.7)
Routing:
- net Net-(JP1-A): track 9.53 -> 12.7 mm
- net GND: vias 149 -> 148
Other:
- board text added: "常時ON"
